File: Hardware/PCB/TMS1mmX19/TMS1mm1chip.kicad_pcb (KiCad board)
At the start: 4 copper layers, 4 parts, among them U0 TMS1mmAout1or2

Commit message: First production-ready PCB/TMS1mmX19
Routing:
- net /SDM_VDD_Shield: track 2.84 -> 5.95 mm
- net /LVDS_VREF: track 3.01 -> 6.09 mm
- net /GND_NMOSI: track 4.90 -> 6.86 mm
- net /Gring: track 2.37 -> 4.14 mm
- net /Ref3: track 4.45 -> 5.16 mm
- net /GND_VREF: track 1.22 -> 1.93 mm
- net /Ref1: track 1.39 -> 2.08 mm
- net /DAC_BufferX2_VREF: track 4.44 -> 5.10 mm
Other:
- copper layers 4 -> 16
Changed lines of the file:
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@@
-(kicad_pcb (version 20170123) (host pcbnew "(2017-07-14 revision 4082470c1)-master")
+(kicad_pcb (version 20170123) (host pcbnew "(2017-07-14 revision d3b382c28)-master")
   (general
-    (thickness 1.6)
+    (thickness 1.92024)
     (drawings 0)
-    (tracks 190)
+    (tracks 205)
     (zones 0)
     (modules 4)
@@
   (layers
     (0 F.Cu signal)
-    (1 In1.Cu power)
-    (2 In2.Cu jumper)
+    (1 In1.Cu signal)
+    (2 In2.Cu signal)
+    (3 In3.Cu signal)
+    (4 In4.Cu signal)
+    (5 In5.Cu signal)
+    (6 In6.Cu signal)
+    (7 In7.Cu signal)
+    (8 In8.Cu signal)
+    (9 In9.Cu signal)
+    (10 In10.Cu signal)
+    (11 In11.Cu signal)
+    (12 In12.Cu signal)
+    (13 In13.Cu signal)
+    (14 In14.Cu signal)
     (31 B.Cu signal)
+    (32 B.Adhes user)
     (33 F.Adhes user)
     (34 B.Paste user)
@@
     (uvia_dia 0.3048)
     (uvia_drill 0.1016)
-    (diff_pair_gap 0.2032)
+    (diff_pair_gap 0.1778)
     (diff_pair_width 0.1016)
     (add_net /AGND)
@@
     )
   )
+  (segment (start 139.7 107.055625) (end 137.927375 107.055625) (width 0.1016) (layer In3.Cu) (net 1))
   (segment (start 137.44 107.322325) (end 137.6686 107.322325) (width 0.1016) (layer F.Cu) (net 1) (status 10))
   (segment (start 137.6686 107.322325) (end 137.9353 107.055625) (width 0.1016) (layer F.Cu) (net 1))
@@
   (segment (start 140.131801 107.487424) (end 139.979399 107.639826) (width 0.1016) (layer F.Cu) (net 3))
   (segment (start 141.96 107.576325) (end 141.96 107.322325) (width 0.1016) (layer F.Cu) (net 3) (status 30))
+  (segment (start 139.24817 104.8766) (end 137.922 104.8766) (width 0.1016) (layer In2.Cu) (net 4))
+  (segment (start 139.7 105.32843) (end 139.24817 104.8766) (width 0.1016) (layer In2.Cu) (net 4))
   (segment (start 138.840465 106.623821) (end 139.268199 106.196087) (width 0.1016) (layer F.Cu) (net 4))
   (segment (start 136.8304 107.703325) (end 136.6018 107.703325) (width 0.1016) (layer F.Cu) (net 4) (status 10))
@@
   (segment (start 136.8304 108.97333) (end 136.635182 108.97333) (width 0.1016) (layer F.Cu) (net 10) (status 10))
   (segment (start 136.635182 108.97333) (end 136.347211 108.685359) (width 0.1016) (layer F.Cu) (net 10))
+  (segment (start 138.9888 107.061) (end 137.922 107.061) (width 0.1016) (layer In6.Cu) (net 11))
+  (segment (start 139.1666 107.2388) (end 138.9888 107.061) (width 0.1016) (layer In6.Cu) (net 11))
+  (segment (start 139.1666 108.249425) (end 139.1666 107.2388) (width 0.1016) (layer In6.Cu) (net 11))
+  (segment (start 139.7 108.782825) (end 139.1666 108.249425) (width 0.1016) (layer In6.Cu) (net 11))
   (segment (start 138.425935 108.173224) (end 139.090399 108.173224) (width 0.1016) (layer F.Cu) (net 11))
   (segment (start 138.201411 108.397748) (end 138.425935 108.173224) (width 0.1016) (layer F.Cu) (net 11))
@@
   (segment (start 142.214 108.338325) (end 142.341 108.211325) (width 0.1016) (layer F.Cu) (net 22))
   (segment (start 141.96 108.338325) (end 142.214 108.338325) (width 0.1016) (layer F.Cu) (net 22) (status 10))
+  (segment (start 140.7668 105.43003) (end 141.42183 105.43003) (width 0.1016) (layer In2.Cu) (net 23))
   (segment (start 140.7668 105.43003) (end 141.269127 105.43003) (width 0.1016) (layer F.Cu) (net 23) (status 10))
   (segment (start 141.269127 105.43003) (end 142.849001 107.009904) (width 0.1016) (layer F.Cu) (net 23))
@@
   (segment (start 142.5696 109.22733) (end 142.5061 109.22733) (width 0.1016) (layer F.Cu) (net 25) (status 30))
   (segment (start 142.5061 109.22733) (end 142.163199 108.884429) (width 0.1016) (layer F.Cu) (net 25) (status 10))
+  (segment (start 140.7668 108.884425) (end 141.457975 108.884425) (width 0.1016) (layer In6.Cu) (net 26))
   (segment (start 141.7314 109.35433) (end 141.96 109.35433) (width 0.1016) (layer F.Cu) (net 26) (status 20))
   (segment (start 141.236705 109.35433) (end 141.7314 109.35433) (width 0.1016) (layer F.Cu) (net 26))
   (segment (start 140.7668 108.884425) (end 141.236705 109.35433) (width 0.1016) (layer F.Cu) (net 26) (status 10))
+  (segment (start 140.7668 106.52223) (end 141.47263 106.52223) (width 0.1016) (layer In3.Cu) (net 27))
   (segment (start 141.6558 108.498947) (end 141.6558 107.41123) (width 0.1016) (layer F.Cu) (net 27))
   (segment (start 141.6558 107.41123) (end 140.7668 106.52223) (width 0.1016) (layer F.Cu) (net 27) (status 20))
@@
   (segment (start 142.488318 108.681226) (end 141.838079 108.681226) (width 0.1016) (layer F.Cu) (net 27))
   (segment (start 141.838079 108.681226) (end 141.6558 108.498947) (width 0.1016) (layer F.Cu) (net 27))
+  (segment (start 140.7668 109.67182) (end 141.47262 109.67182) (width 0.1016) (layer In5.Cu) (net 28))
   (segment (start 140.7668 109.67182) (end 141.161931 109.67182) (width 0.1016) (layer F.Cu) (net 28) (status 10))
   (segment (start 141.225421 109.60833) (end 141.7314 109.60833) (width 0.1016) (layer F.Cu) (net 28))
@@
   (segment (start 142.3156 109.73533) (end 142.341 109.73533) (width 0.1016) (layer F.Cu) (net 29))
   (segment (start 142.341 109.73533) (end 142.5696 109.73533) (width 0.1016) (layer F.Cu) (net 29) (status 20))
+  (segment (start 140.1318 112.776) (end 137.922 112.776) (width 0.1016) (layer In5.Cu) (net 30))
+  (segment (start 140.487401 112.420399) (end 140.1318 112.776) (width 0.1016) (layer In5.Cu) (net 30))
+  (segment (start 140.7668 112.13562) (end 140.487401 112.415019) (width 0.1016) (layer In5.Cu) (net 30))
+  (segment (start 140.487401 112.415019) (end 140.487401 112.420399) (width 0.1016) (layer In5.Cu) (net 30))
   (segment (start 142.5702 110.6678) (end 141.381779 111.856221) (width 0.1016) (layer F.Cu) (net 30))
   (segment (start 141.381779 111.856221) (end 141.046199 111.856221) (width 0.1016) (layer F.Cu) (net 30))
